Commit message: made changes to urdf and launch file to see robot

File: nuturtle_description/urdf/turtlebot3_burger.gazebo.xacro (robot description, xacro)
@@ -13,5 +13,5 @@
           <preserveFixedJoint>true</preserveFixedJoint>
         </gazebo>
-        <gazebo reference="base_laser" >
+        <gazebo reference="base_scan" >
           <sensor name='gpu_lidar' type='gpu_lidar'>
             <topic>scan</topic>
@@ -40,5 +40,5 @@
             <alwaysOn>1</alwaysOn>
             <visualize>true</visualize>
-            <ignition_frame_id>base_laser</ignition_frame_id>
+            <ignition_frame_id>base_scan</ignition_frame_id>
         </sensor>
     </gazebo>

File: nuturtle_description/urdf/turtlebot3_burger.urdf.xacro (robot description, xacro)
@@ -44,5 +44,23 @@
     <color rgba="1.0 1.0 1.0 1.0"/>
   </material>
-  <link name="base_footprint"/>
+  <link name="base_footprint">
+    <visual>
+      <origin xyz="0 0 0" rpy="0 0 0"/>
+      <geometry>
+        <cylinder radius="0.02" length="0.001"/>
+      </geometry>
+    </visual>
+    <collision>
+      <origin xyz="0 0 0" rpy="0 0 0"/>
+      <geometry>
+        <cylinder radius="0.1" length="0.05"/>
+      </geometry>
+    </collision>
+    <inertial>
+      <mass value="1.0"/>
+      <origin xyz="0 0 0" rpy="0 0 0"/>
+      <inertia ixx="0.00001" ixy="0.0" ixz="0.0" iyy="0.00001" iyz="0.0" izz="0.00001"/>
+    </inertial>
+  </link>
   <joint name="base_joint" type="fixed">
     <parent link="base_footprint"/>

Commit message: fixed joint issue and missing base footprint still throws mesh errors

File: nuturtle_description/urdf/turtlebot3_burger.gazebo.xacro (robot description, xacro)
@@ -49,6 +49,6 @@
         <left_joint>wheel_left_joint</left_joint>
         <right_joint>wheel_right_joint</right_joint>
-        <wheel_separation>"${track_width}"</wheel_separation>
-        <wheel_radius>"${wheel_radius}"</wheel_radius>
+        <wheel_separation>0.16</wheel_separation>
+        <wheel_radius>0.033</wheel_radius>
         <odom_publish_frequency>30</odom_publish_frequency>
         <frame_id>odom</frame_id>

File: nuturtle_description/urdf/turtlebot3_burger.urdf.xacro (robot description, xacro)
@@ -64,6 +64,6 @@
   </link>
   <joint name="base_joint" type="fixed">
-    <parent link="base_footprint"/>
-    <child link="base_link"/>
+    <parent link="base_link"/>
+    <child link="base_footprint"/>
     <origin xyz="0.0 0.0 0.010" rpy="0 0 0"/>
   </joint>
